File: pcbDesign/ATSAME51J18A-devboard-panel.kicad_pcb (KiCad board)
At the start: 2 copper layers, 100 x 100 mm, 273 parts, among them IC1 MP9361DJ-LF-P, J1 Micro_SD_Card, J10 CAN, J11 Conn_01x32_Male, J2 USB C, J3 QWIIC, J4 S2B-PH-K-S(LF)(SN), J7 Conn_01x32_Male, SW1 RST, U1 TCAN1051GVDRQ1, U2 ATSAME51J18A-A, U3 MIC5219-5.0YMM, U4 LM27762, U5 TPS60501DGS, U7 BQ24074RGT, U8 BQ27441DRZR-G1B, Y1 32.768

Commit message: Panelised prototype(v0.2)
Parts:
- removed the C1 at (123.2, 133.5)
- removed the C1 at (123.2, 102.0)
- removed the C1 at (123.2, 70.6)
- removed the C10 at (113.0, 122.3)
- removed the C10 at (113.0, 90.8)
- removed the C10 at (113.0, 59.4)
- removed the C11 at (99.8, 130.2)
- removed the C11 at (99.8, 98.7)
- removed the C11 at (99.8, 67.3)
- removed the C12 at (79.5, 134.5)
- removed the C12 at (79.5, 103.0)
- removed the C12 at (79.5, 71.6)
- removed the C13 at (99.7, 128.9)
- removed the C13 at (99.7, 97.5)
- removed the C13 at (99.7, 66.0)
- removed the C14 at (109.7, 124.3)
- removed the C14 at (109.7, 92.9)
- removed the C14 at (109.7, 61.4)
- removed the C15 at (107.9, 131.4)
- removed the C15 at (107.9, 100.0)
- removed the C15 at (107.9, 68.5)
- removed the C16 at (104.1, 124.7)
- removed the C16 at (104.1, 93.3)
- removed the C16 at (104.1, 61.8)
- removed the C17 at (99.8, 122.2)
- removed the C17 at (99.8, 90.7)
- removed the C17 at (99.8, 59.3)
- removed the C18 at (112.7, 128.6)
- removed the C18 at (112.7, 97.2)
- removed the C18 at (112.7, 65.7)
- removed the C19 at (107.4, 123.8)
- removed the C19 at (107.4, 92.4)
- removed the C19 at (107.4, 60.9)
- removed the C2 at (121.9, 123.3)
- removed the C2 at (121.9, 91.9)
- removed the C2 at (121.9, 60.4)
- removed the C20 at (102.3, 119.0)
- removed the C20 at (102.3, 87.5)
- removed the C20 at (102.3, 56.1)
- removed the C21 at (107.2, 121.0)
- removed the C21 at (107.2, 89.6)
- removed the C21 at (107.2, 58.1)
- removed the C22 at (66.4, 130.5)
- removed the C22 at (66.4, 99.1)
- removed the C22 at (66.4, 67.7)
- removed the C23 at (66.4, 122.5)
- removed the C23 at (66.4, 91.1)
- removed the C23 at (66.4, 59.7)
- removed the C24 at (73.1, 129.7)
- removed the C24 at (73.1, 98.2)
- removed the C24 at (73.1, 66.8)
- removed the C3 at (84.3, 135.1)
- removed the C3 at (84.3, 103.6)
- removed the C3 at (84.3, 72.2)
- removed the C4 at (84.3, 131.3)
- removed the C4 at (84.3, 99.8)
- removed the C4 at (84.3, 68.4)
- removed the C8 at (76.9, 132.5)
- removed the C8 at (76.9, 101.0)
- removed the C8 at (76.9, 69.6)
- removed the C9 at (106.8, 129.5)
- removed the C9 at (106.8, 98.1)
- removed the C9 at (106.8, 66.6)
- removed the D1 at (113.8, 122.5)
- removed the D1 at (113.8, 91.1)
- removed the D1 at (113.8, 59.7)
- removed the D2 at (61.7, 126.4)
- removed the D2 at (61.7, 94.9)
- removed the D2 at (61.7, 63.5)
- removed the D3 at (71.0, 132.3)
- removed the D3 at (71.0, 100.9)
- removed the D3 at (71.0, 69.4)
- removed the D4 at (61.7, 128.6)
- removed the D4 at (61.7, 97.2)
- removed the D4 at (61.7, 65.7)
- removed the D5 at (100.3, 134.0)
- removed the D5 at (100.3, 102.5)
- removed the D5 at (100.3, 71.1)
- removed the D6 at (68.0, 131.2)
- removed the D6 at (68.0, 99.7)
- removed the D6 at (68.0, 68.3)
- removed the G*** at (73.1, 127.4)
- removed the G*** at (73.1, 95.9)
- removed the G*** at (73.1, 64.5)
- removed the IC1 at (111.7, 125.1)
- removed the IC1 at (111.7, 93.6)
- removed the IC1 at (111.7, 62.2)
- removed the J1 at (125.4, 127.1)
- removed the J1 at (125.4, 95.7)
- removed the J1 at (125.4, 64.2)
- removed the J10 at (127.2, 123.3)
- removed the J10 at (127.2, 91.9)
- removed the J10 at (127.2, 60.4)
- removed the J2 at (54.8, 130.4)
- removed the J2 at (54.8, 99.0)
- removed the J2 at (54.8, 67.5)
- removed the J3 at (127.2, 130.9)
- removed the J3 at (127.2, 99.5)
- removed the J3 at (127.2, 68.0)
- removed the J4 at (56.4, 121.3)
- removed the J4 at (56.4, 89.8)
- removed the J4 at (56.4, 58.4)
- removed the R1 at (61.7, 129.9)
- removed the R1 at (61.7, 98.5)
- removed the R1 at (61.7, 67.0)
- removed the R10 at (106.6, 127.6)
- removed the R10 at (106.6, 96.2)
- removed the R10 at (106.6, 64.7)
- removed the R11 at (63.2, 128.6)
- removed the R11 at (63.2, 97.2)
- removed the R11 at (63.2, 65.7)
- removed the R12 at (65.1, 130.5)
- removed the R12 at (65.1, 99.1)
- removed the R12 at (65.1, 67.7)
- removed the R13 at (63.2, 123.6)
- removed the R13 at (63.2, 92.1)
- removed the R13 at (63.2, 60.7)
- removed the R14 at (74.8, 126.4)
- removed the R14 at (74.8, 94.9)
- removed the R14 at (74.8, 63.5)
- removed the R15 at (74.8, 127.9)
- removed the R15 at (74.8, 96.4)
- removed the R15 at (74.8, 65.0)
- removed the R16 at (70.1, 121.8)
- removed the R16 at (70.1, 90.3)
- removed the R16 at (70.1, 58.9)
- removed the R17 at (74.9, 121.8)
- removed the R17 at (74.9, 90.3)
- removed the R17 at (74.9, 58.9)
- removed the R18 at (74.9, 123.1)
- removed the R18 at (74.9, 91.6)
- removed the R18 at (74.9, 60.2)
- removed the R2 at (54.1, 130.4)
- removed the R2 at (54.1, 99.0)
- removed the R2 at (54.1, 67.5)
- removed the R20 at (70.3, 130.4)
- removed the R20 at (70.3, 99.0)
- removed the R20 at (70.3, 67.5)
- removed the R21 at (71.0, 129.2)
- removed the R21 at (71.0, 97.7)
- removed the R21 at (71.0, 66.3)
- removed the R22 at (67.7, 122.5)
- removed the R22 at (67.7, 91.1)
- removed the R22 at (67.7, 59.7)
- removed the R4 at (77.4, 124.6)
- removed the R4 at (77.4, 93.1)
- removed the R4 at (77.4, 61.7)
- removed the R5 at (104.4, 132.5)
- removed the R5 at (104.4, 101.0)
- removed the R5 at (104.4, 69.6)
- removed the R6 at (101.6, 132.7)
- removed the R6 at (101.6, 101.3)
- removed the R6 at (101.6, 69.8)
- removed the R7 at (106.8, 131.4)
- removed the R7 at (106.8, 100.0)
- removed the R7 at (106.8, 68.5)
- removed the R8 at (104.1, 126.0)
- removed the R8 at (104.1, 94.5)
- removed the R8 at (104.1, 63.1)
- removed the R9 at (106.8, 133.3)
- removed the R9 at (106.8, 101.9)
- removed the R9 at (106.8, 70.4)
- removed the REF** at (134.7, 125.6)
- removed the REF** at (134.7, 95.2)
- removed the REF** at (134.7, 96.2)
- removed the REF** at (134.7, 97.2)
- removed the REF** at (49.4, 97.2)
- removed the REF** at (49.4, 96.2)
- removed the REF** at (49.4, 95.2)
- removed the REF** at (49.4, 94.2)
- removed the REF** at (134.7, 62.7)
- removed the REF** at (134.7, 63.7)
- removed the REF** at (134.7, 64.7)
- removed the REF** at (134.7, 126.6)
- removed the REF** at (134.7, 65.7)
- removed the REF** at (49.4, 65.7)
- removed the REF** at (49.4, 64.7)
- removed the REF** at (49.4, 63.7)
- removed the REF** at (49.4, 62.7)
- removed the REF** at (93.5, 141.9)
- removed the REF** at (92.5, 141.9)
- removed the REF** at (91.5, 141.9)
- removed the REF** at (90.5, 141.9)
- removed the REF** at (90.5, 112.3)
- removed the REF** at (134.7, 127.6)
- removed the REF** at (91.5, 112.3)
- removed the REF** at (92.5, 112.3)
- removed the REF** at (93.5, 112.3)
- removed the REF** at (93.5, 110.5)
- removed the REF** at (92.5, 110.5)
- removed the REF** at (91.5, 110.5)
- removed the REF** at (90.5, 110.5)
- removed the REF** at (90.5, 80.8)
- removed the REF** at (91.5, 80.8)
- removed the REF** at (92.5, 80.8)
- removed the REF** at (134.7, 128.6)
- removed the REF** at (93.5, 80.8)
- removed the REF** at (93.5, 79.0)
- removed the REF** at (92.5, 79.0)
- removed the REF** at (91.5, 79.0)
- removed the REF** at (90.5, 79.0)
- removed the REF** at (90.5, 49.4)
- removed the REF** at (91.5, 49.4)
- removed the REF** at (92.5, 49.4)
- removed the REF** at (93.5, 49.4)
- removed the REF** at (49.4, 128.6)
- removed the REF** at (49.4, 127.6)
- removed the REF** at (49.4, 126.6)
- removed the REF** at (49.4, 125.6)
- removed the REF** at (134.7, 94.2)
- removed the SW1 at (111.5, 129.9)
- removed the SW1 at (111.5, 98.5)
- removed the SW1 at (111.5, 67.0)
- removed the U3 at (79.8, 129.9)
- removed the U3 at (79.8, 98.5)
- removed the U3 at (79.8, 67.0)
- removed the U4 at (103.5, 129.5)
- removed the U4 at (103.5, 98.1)
- removed the U4 at (103.5, 66.6)
- removed the U5 at (103.3, 121.3)
- removed the U5 at (103.3, 89.8)
- removed the U5 at (103.3, 58.4)
- removed the U7 at (66.4, 126.4)
- removed the U7 at (66.4, 94.9)
- removed the U7 at (66.4, 63.5)
- removed the U8 at (71.2, 125.2)
- removed the U8 at (71.2, 93.8)
- removed the U8 at (71.2, 62.3)
- removed the Y1 at (83.7, 133.2)
- removed the Y1 at (83.7, 101.7)
- removed the Y1 at (83.7, 70.3)
- added C1: 100n, Capacitor_SMD:C_0402_1005Metric, F.Cu at (123.2, 122.8)
- added C1: 100n, Capacitor_SMD:C_0402_1005Metric, F.Cu at (123.2, 91.4)
- added C1: 100n, Capacitor_SMD:C_0402_1005Metric, F.Cu at (123.2, 59.9)
- added C10: 2.2u, Capacitor_SMD:C_0402_1005Metric, F.Cu at (116.8, 131.2)
- added C10: 2.2u, Capacitor_SMD:C_0402_1005Metric, F.Cu at (116.8, 99.7)
- added C10: 2.2u, Capacitor_SMD:C_0402_1005Metric, F.Cu at (116.8, 68.3)
- added C11: 4.7u, Capacitor_SMD:C_0402_1005Metric, F.Cu at (103.6, 123.3)
- added C11: 4.7u, Capacitor_SMD:C_0402_1005Metric, F.Cu at (103.6, 91.9)
- added C11: 4.7u, Capacitor_SMD:C_0402_1005Metric, F.Cu at (103.6, 60.4)
- added C12: 2.2u, Capacitor_SMD:C_0402_1005Metric, F.Cu at (80.5, 120.3)
- added C12: 2.2u, Capacitor_SMD:C_0402_1005Metric, F.Cu at (80.5, 88.8)
- added C12: 2.2u, Capacitor_SMD:C_0402_1005Metric, F.Cu at (80.5, 57.4)
- added C13: 4.7u, Capacitor_SMD:C_0402_1005Metric, F.Cu at (103.5, 124.6)
- added C13: 4.7u, Capacitor_SMD:C_0402_1005Metric, F.Cu at (103.5, 93.1)
- added C13: 4.7u, Capacitor_SMD:C_0402_1005Metric, F.Cu at (103.5, 61.7)
- added C14: 0.47u, Capacitor_SMD:C_0402_1005Metric, F.Cu at (113.5, 129.2)
- added C14: 0.47u, Capacitor_SMD:C_0402_1005Metric, F.Cu at (113.5, 97.7)
- added C14: 0.47u, Capacitor_SMD:C_0402_1005Metric, F.Cu at (113.5, 66.3)
- added C15: 2.2u, Capacitor_SMD:C_0402_1005Metric, F.Cu at (111.7, 122.0)
- added C15: 2.2u, Capacitor_SMD:C_0402_1005Metric, F.Cu at (111.7, 90.6)
- added C15: 2.2u, Capacitor_SMD:C_0402_1005Metric, F.Cu at (111.7, 59.1)
- added C16: 2.2u, Capacitor_SMD:C_0402_1005Metric, F.Cu at (107.9, 128.8)
- added C16: 2.2u, Capacitor_SMD:C_0402_1005Metric, F.Cu at (107.9, 97.3)
- added C16: 2.2u, Capacitor_SMD:C_0402_1005Metric, F.Cu at (107.9, 65.9)
- added C17: 1u, Capacitor_SMD:C_0402_1005Metric, F.Cu at (103.6, 131.3)
- added C17: 1u, Capacitor_SMD:C_0402_1005Metric, F.Cu at (103.6, 99.9)
- added C17: 1u, Capacitor_SMD:C_0402_1005Metric, F.Cu at (103.6, 68.4)
- added C18: 10u, Capacitor_SMD:C_0402_1005Metric, F.Cu at (116.5, 124.8)
- added C18: 10u, Capacitor_SMD:C_0402_1005Metric, F.Cu at (116.5, 93.4)
- added C18: 10u, Capacitor_SMD:C_0402_1005Metric, F.Cu at (116.5, 61.9)
- added C19: 4.7u, Capacitor_SMD:C_0402_1005Metric, F.Cu at (111.2, 129.7)
- added C19: 4.7u, Capacitor_SMD:C_0402_1005Metric, F.Cu at (111.2, 98.2)
- added C19: 4.7u, Capacitor_SMD:C_0402_1005Metric, F.Cu at (111.2, 66.8)
- added C2: 100n, Capacitor_SMD:C_0402_1005Metric, F.Cu at (121.9, 133.0)
- added C2: 100n, Capacitor_SMD:C_0402_1005Metric, F.Cu at (121.9, 101.5)
- added C2: 100n, Capacitor_SMD:C_0402_1005Metric, F.Cu at (121.9, 70.1)
- added C20: 22u, Capacitor_SMD:C_0402_1005Metric, F.Cu at (106.1, 134.5)
- added C20: 22u, Capacitor_SMD:C_0402_1005Metric, F.Cu at (106.1, 103.0)
- added C20: 22u, Capacitor_SMD:C_0402_1005Metric, F.Cu at (106.1, 71.6)
- added C21: 1u, Capacitor_SMD:C_0402_1005Metric, F.Cu at (111.0, 132.5)
- added C21: 1u, Capacitor_SMD:C_0402_1005Metric, F.Cu at (111.0, 101.0)
- added C21: 1u, Capacitor_SMD:C_0402_1005Metric, F.Cu at (111.0, 69.6)
- added C22: 4.7u, Capacitor_SMD:C_0402_1005Metric, F.Cu at (67.7, 126.7)
- added C22: 4.7u, Capacitor_SMD:C_0402_1005Metric, F.Cu at (67.7, 95.3)
- added C22: 4.7u, Capacitor_SMD:C_0402_1005Metric, F.Cu at (67.7, 63.8)
- added C23: 4.7u, Capacitor_SMD:C_0402_1005Metric, F.Cu at (67.7, 134.7)
- added C23: 4.7u, Capacitor_SMD:C_0402_1005Metric, F.Cu at (67.7, 103.3)
- added C23: 4.7u, Capacitor_SMD:C_0402_1005Metric, F.Cu at (67.7, 71.8)
- added C24: 0.47u, Capacitor_SMD:C_0402_1005Metric, F.Cu at (74.1, 125.1)
- added C24: 0.47u, Capacitor_SMD:C_0402_1005Metric, F.Cu at (74.1, 93.6)
- added C24: 0.47u, Capacitor_SMD:C_0402_1005Metric, F.Cu at (74.1, 62.2)
- added C3: 22u, Capacitor_SMD:C_0402_1005Metric, F.Cu at (81.2, 129.6)
- added C3: 22u, Capacitor_SMD:C_0402_1005Metric, F.Cu at (81.2, 98.1)
- added C3: 22u, Capacitor_SMD:C_0402_1005Metric, F.Cu at (81.2, 66.7)
- added C4: 22u, Capacitor_SMD:C_0402_1005Metric, F.Cu at (81.2, 133.4)
- added C4: 22u, Capacitor_SMD:C_0402_1005Metric, F.Cu at (81.2, 101.9)
- added C4: 22u, Capacitor_SMD:C_0402_1005Metric, F.Cu at (81.2, 70.5)
- added C8: 0.47u, Capacitor_SMD:C_0402_1005Metric, F.Cu at (77.9, 122.3)
- added C8: 0.47u, Capacitor_SMD:C_0402_1005Metric, F.Cu at (77.9, 90.8)
- added C8: 0.47u, Capacitor_SMD:C_0402_1005Metric, F.Cu at (77.9, 59.4)
- added C9: 0.47u, Capacitor_SMD:C_0402_1005Metric, F.Cu at (110.6, 123.9)
- added C9: 0.47u, Capacitor_SMD:C_0402_1005Metric, F.Cu at (110.6, 92.5)
- added C9: 0.47u, Capacitor_SMD:C_0402_1005Metric, F.Cu at (110.6, 61.0)
- added D1: WS2812B, LED_SMD:LED_WS2812B_PLCC4_5.0x5.0mm_P3.2mm, F.Cu at (66.0, 121.3)
- added D1: WS2812B, LED_SMD:LED_WS2812B_PLCC4_5.0x5.0mm_P3.2mm, F.Cu at (66.0, 89.8)
- added D1: WS2812B, LED_SMD:LED_WS2812B_PLCC4_5.0x5.0mm_P3.2mm, F.Cu at (66.0, 58.4)
- added D2: D_Schottky, Diode_SMD:D_0402_1005Metric, F.Cu at (61.7, 126.9)
- added D2: D_Schottky, Diode_SMD:D_0402_1005Metric, F.Cu at (61.7, 95.4)
- added D2: D_Schottky, Diode_SMD:D_0402_1005Metric, F.Cu at (61.7, 64.0)
- added D3: D_Schottky, Diode_SMD:D_0402_1005Metric, F.Cu at (74.1, 123.1)
- added D3: D_Schottky, Diode_SMD:D_0402_1005Metric, F.Cu at (74.1, 91.6)
- added D3: D_Schottky, Diode_SMD:D_0402_1005Metric, F.Cu at (74.1, 60.2)
- added D4: D_Schottky, Diode_SMD:D_0402_1005Metric, F.Cu at (61.7, 129.2)
- added D4: D_Schottky, Diode_SMD:D_0402_1005Metric, F.Cu at (61.7, 97.7)
- added D4: D_Schottky, Diode_SMD:D_0402_1005Metric, F.Cu at (61.7, 66.3)
- added D5: D_Schottky, Diode_SMD:D_0402_1005Metric, F.Cu at (102.1, 119.5)
- added D5: D_Schottky, Diode_SMD:D_0402_1005Metric, F.Cu at (102.1, 88.1)
- added D5: D_Schottky, Diode_SMD:D_0402_1005Metric, F.Cu at (102.1, 56.6)
- added D6: D_Schottky, Diode_SMD:D_0402_1005Metric, F.Cu at (69.8, 126.1)
- added D6: D_Schottky, Diode_SMD:D_0402_1005Metric, F.Cu at (69.8, 94.7)
- added D6: D_Schottky, Diode_SMD:D_0402_1005Metric, F.Cu at (69.8, 63.2)
- added G***: LOGO, Symbol:BatonLogo, B.Cu at (93.7, 126.6)
- added G***: LOGO, Symbol:BatonLogo, B.Cu at (93.7, 95.2)
- added G***: LOGO, Symbol:BatonLogo, B.Cu at (93.7, 63.7)
- added IC1: MP9361DJ-LF-P, SamacSys_Parts:SOT95P280X100-6N, F.Cu at (115.5, 128.4)
- added IC1: MP9361DJ-LF-P, SamacSys_Parts:SOT95P280X100-6N, F.Cu at (115.5, 96.9)
- added IC1: MP9361DJ-LF-P, SamacSys_Parts:SOT95P280X100-6N, F.Cu at (115.5, 65.5)
- added J1: Micro_SD_Card, Connector_Card:microSD_HC_Hirose_DM3D-SF, F.Cu at (132.8, 127.1)
- added J1: Micro_SD_Card, Connector_Card:microSD_HC_Hirose_DM3D-SF, F.Cu at (132.8, 95.7)
- added J1: Micro_SD_Card, Connector_Card:microSD_HC_Hirose_DM3D-SF, F.Cu at (132.8, 64.2)
- added J10: CAN, SM04B-SRSS-TB_LF__SN_:JST_SM04B-SRSS-TB(LF)(SN), F.Cu at (136.1, 118.7)
- added J10: CAN, SM04B-SRSS-TB_LF__SN_:JST_SM04B-SRSS-TB(LF)(SN), F.Cu at (136.1, 87.3)
- added J10: CAN, SM04B-SRSS-TB_LF__SN_:JST_SM04B-SRSS-TB(LF)(SN), F.Cu at (136.1, 55.8)
- added J2: USB C, usb_c:12401598E4-2A, F.Cu at (54.8, 130.9)
- added J2: USB C, usb_c:12401598E4-2A, F.Cu at (54.8, 99.5)
- added J2: USB C, usb_c:12401598E4-2A, F.Cu at (54.8, 68.0)
- added J3: QWIIC, SM04B-SRSS-TB_LF__SN_:JST_SM04B-SRSS-TB(LF)(SN), F.Cu at (136.1, 135.5)
- added J3: QWIIC, SM04B-SRSS-TB_LF__SN_:JST_SM04B-SRSS-TB(LF)(SN), F.Cu at (136.1, 104.1)
- added J3: QWIIC, SM04B-SRSS-TB_LF__SN_:JST_SM04B-SRSS-TB(LF)(SN), F.Cu at (136.1, 72.6)
- added J4: S2B-PH-K-S(LF)(SN), S2B-PH-K-S_LF__SN_:JST_S2B-PH-K-S(LF)(SN), F.Cu at (56.4, 121.8)
- added J4: S2B-PH-K-S(LF)(SN), S2B-PH-K-S_LF__SN_:JST_S2B-PH-K-S(LF)(SN), F.Cu at (56.4, 90.3)
- added J4: S2B-PH-K-S(LF)(SN), S2B-PH-K-S_LF__SN_:JST_S2B-PH-K-S(LF)(SN), F.Cu at (56.4, 58.9)
- added R1: 5.1k, Resistor_SMD:R_0402_1005Metric, F.Cu at (61.7, 130.4)
- added R1: 5.1k, Resistor_SMD:R_0402_1005Metric, F.Cu at (61.7, 99.0)
- added R1: 5.1k, Resistor_SMD:R_0402_1005Metric, F.Cu at (61.7, 67.5)
- added R10: 50k, Resistor_SMD:R_0402_1005Metric, F.Cu at (110.5, 125.9)
- added R10: 50k, Resistor_SMD:R_0402_1005Metric, F.Cu at (110.5, 94.4)
- added R10: 50k, Resistor_SMD:R_0402_1005Metric, F.Cu at (110.5, 63.0)
- added R11: 46.4k, Resistor_SMD:R_0402_1005Metric, F.Cu at (65.0, 128.6)
- added R11: 46.4k, Resistor_SMD:R_0402_1005Metric, F.Cu at (65.0, 97.2)
- added R11: 46.4k, Resistor_SMD:R_0402_1005Metric, F.Cu at (65.0, 65.7)
- added R12: 1.18k, Resistor_SMD:R_0402_1005Metric, F.Cu at (66.4, 126.7)
- added R12: 1.18k, Resistor_SMD:R_0402_1005Metric, F.Cu at (66.4, 95.3)
- added R12: 1.18k, Resistor_SMD:R_0402_1005Metric, F.Cu at (66.4, 63.8)
- added R13: 1.13k, Resistor_SMD:R_0402_1005Metric, F.Cu at (65.0, 133.7)
- added R13: 1.13k, Resistor_SMD:R_0402_1005Metric, F.Cu at (65.0, 102.3)
- added R13: 1.13k, Resistor_SMD:R_0402_1005Metric, F.Cu at (65.0, 70.8)
- added R14: 5.1k, Resistor_SMD:R_0402_1005Metric, F.Cu at (75.8, 128.4)
- added R14: 5.1k, Resistor_SMD:R_0402_1005Metric, F.Cu at (75.8, 96.9)
- added R14: 5.1k, Resistor_SMD:R_0402_1005Metric, F.Cu at (75.8, 65.5)
- added R15: 5.1k, Resistor_SMD:R_0402_1005Metric, F.Cu at (75.8, 126.9)
- added R15: 5.1k, Resistor_SMD:R_0402_1005Metric, F.Cu at (75.8, 95.4)
- added R15: 5.1k, Resistor_SMD:R_0402_1005Metric, F.Cu at (75.8, 64.0)
- added R16: 0.01, Resistor_SMD:R_0402_1005Metric, F.Cu at (71.1, 133.0)
- added R16: 0.01, Resistor_SMD:R_0402_1005Metric, F.Cu at (71.1, 101.5)
- added R16: 0.01, Resistor_SMD:R_0402_1005Metric, F.Cu at (71.1, 70.1)
- added R17: 10k, Resistor_SMD:R_0402_1005Metric, F.Cu at (75.9, 133.0)
- added R17: 10k, Resistor_SMD:R_0402_1005Metric, F.Cu at (75.9, 101.5)
- added R17: 10k, Resistor_SMD:R_0402_1005Metric, F.Cu at (75.9, 70.1)
- added R18: 10k, Resistor_SMD:R_0402_1005Metric, F.Cu at (75.9, 131.7)
- added R18: 10k, Resistor_SMD:R_0402_1005Metric, F.Cu at (75.9, 100.2)
- added R18: 10k, Resistor_SMD:R_0402_1005Metric, F.Cu at (75.9, 68.8)
- added R2: 5.1k, Resistor_SMD:R_0402_1005Metric, F.Cu at (62.2, 133.5)
- added R2: 5.1k, Resistor_SMD:R_0402_1005Metric, F.Cu at (62.2, 102.0)
- added R2: 5.1k, Resistor_SMD:R_0402_1005Metric, F.Cu at (62.2, 70.6)
- added R20: 10k, Resistor_SMD:R_0402_1005Metric, F.Cu at (71.3, 124.3)
- added R20: 10k, Resistor_SMD:R_0402_1005Metric, F.Cu at (71.3, 92.9)
- added R20: 10k, Resistor_SMD:R_0402_1005Metric, F.Cu at (71.3, 61.4)
- added R21: 10k, Resistor_SMD:R_0402_1005Metric, F.Cu at (72.0, 125.6)
- added R21: 10k, Resistor_SMD:R_0402_1005Metric, F.Cu at (72.0, 94.1)
- added R21: 10k, Resistor_SMD:R_0402_1005Metric, F.Cu at (72.0, 62.7)
- added R22: 10k, Resistor_SMD:R_0402_1005Metric, F.Cu at (68.9, 134.7)
- added R22: 10k, Resistor_SMD:R_0402_1005Metric, F.Cu at (68.9, 103.3)
- added R22: 10k, Resistor_SMD:R_0402_1005Metric, F.Cu at (68.9, 71.8)
- added R4: 10k, Resistor_SMD:R_0402_1005Metric, F.Cu at (78.4, 130.2)
- added R4: 10k, Resistor_SMD:R_0402_1005Metric, F.Cu at (78.4, 98.7)
- added R4: 10k, Resistor_SMD:R_0402_1005Metric, F.Cu at (78.4, 67.3)
- added R5: 10k, Resistor_SMD:R_0402_1005Metric, F.Cu at (108.2, 121.0)
- added R5: 10k, Resistor_SMD:R_0402_1005Metric, F.Cu at (108.2, 89.6)
- added R5: 10k, Resistor_SMD:R_0402_1005Metric, F.Cu at (108.2, 58.1)
- added R6: 10k, Resistor_SMD:R_0402_1005Metric, F.Cu at (105.4, 120.8)
- added R6: 10k, Resistor_SMD:R_0402_1005Metric, F.Cu at (105.4, 89.3)
- added R6: 10k, Resistor_SMD:R_0402_1005Metric, F.Cu at (105.4, 57.9)
- added R7: 87.5k, Resistor_SMD:R_0402_1005Metric, F.Cu at (110.6, 122.0)
- added R7: 87.5k, Resistor_SMD:R_0402_1005Metric, F.Cu at (110.6, 90.6)
- added R7: 87.5k, Resistor_SMD:R_0402_1005Metric, F.Cu at (110.6, 59.1)
- added R8: 87.5k, Resistor_SMD:R_0402_1005Metric, F.Cu at (107.9, 127.5)
- added R8: 87.5k, Resistor_SMD:R_0402_1005Metric, F.Cu at (107.9, 96.1)
- added R8: 87.5k, Resistor_SMD:R_0402_1005Metric, F.Cu at (107.9, 64.6)
- added R9: 50k, Resistor_SMD:R_0402_1005Metric, F.Cu at (110.6, 120.1)
- added R9: 50k, Resistor_SMD:R_0402_1005Metric, F.Cu at (110.6, 88.7)
- added R9: 50k, Resistor_SMD:R_0402_1005Metric, F.Cu at (110.6, 57.2)
- added REF**: NPTH, NPTH, F.Cu at (140.8, 130.4)
- added REF**: NPTH, NPTH, F.Cu at (49.4, 132.4)
- added REF**: NPTH, NPTH, F.Cu at (49.4, 131.4)
- added REF**: NPTH, NPTH, F.Cu at (49.4, 130.4)
- added REF**: NPTH, NPTH, F.Cu at (49.4, 123.9)
- added REF**: NPTH, NPTH, F.Cu at (49.4, 122.9)
- added REF**: NPTH, NPTH, F.Cu at (49.4, 121.9)
- added REF**: NPTH, NPTH, F.Cu at (49.4, 120.9)
- added REF**: NPTH, NPTH, F.Cu at (140.8, 98.9)
- added REF**: NPTH, NPTH, F.Cu at (140.8, 99.9)
- added REF**: NPTH, NPTH, F.Cu at (140.8, 100.9)
- added REF**: NPTH, NPTH, F.Cu at (140.8, 131.4)
- added REF**: NPTH, NPTH, F.Cu at (140.8, 101.9)
- added REF**: NPTH, NPTH, F.Cu at (140.8, 89.4)
- added REF**: NPTH, NPTH, F.Cu at (140.8, 90.4)
- added REF**: NPTH, NPTH, F.Cu at (140.8, 91.4)
- added REF**: NPTH, NPTH, F.Cu at (140.8, 92.4)
- added REF**: NPTH, NPTH, F.Cu at (49.4, 101.9)
- added REF**: NPTH, NPTH, F.Cu at (49.4, 100.9)
- added REF**: NPTH, NPTH, F.Cu at (49.4, 99.9)
- added REF**: NPTH, NPTH, F.Cu at (49.4, 98.9)
- added REF**: NPTH, NPTH, F.Cu at (49.4, 92.4)
- added REF**: NPTH, NPTH, F.Cu at (140.8, 132.4)
- added REF**: NPTH, NPTH, F.Cu at (49.4, 91.4)
- added REF**: NPTH, NPTH, F.Cu at (49.4, 90.4)
- added REF**: NPTH, NPTH, F.Cu at (49.4, 89.4)
- added REF**: NPTH, NPTH, F.Cu at (140.8, 67.5)
- added REF**: NPTH, NPTH, F.Cu at (140.8, 68.5)
- added REF**: NPTH, NPTH, F.Cu at (140.8, 69.5)
- added REF**: NPTH, NPTH, F.Cu at (140.8, 70.5)
- added REF**: NPTH, NPTH, F.Cu at (140.8, 58.0)
- added REF**: NPTH, NPTH, F.Cu at (140.8, 59.0)
- added REF**: NPTH, NPTH, F.Cu at (140.8, 60.0)
- added REF**: NPTH, NPTH, F.Cu at (140.8, 133.4)
- added REF**: NPTH, NPTH, F.Cu at (140.8, 61.0)
- added REF**: NPTH, NPTH, F.Cu at (49.4, 70.5)
- added REF**: NPTH, NPTH, F.Cu at (49.4, 69.5)
- added REF**: NPTH, NPTH, F.Cu at (49.4, 68.5)
- added REF**: NPTH, NPTH, F.Cu at (49.4, 67.5)
- added REF**: NPTH, NPTH, F.Cu at (49.4, 61.0)
- added REF**: NPTH, NPTH, F.Cu at (49.4, 60.0)
- added REF**: NPTH, NPTH, F.Cu at (49.4, 59.0)
- added REF**: NPTH, NPTH, F.Cu at (49.4, 58.0)
- added REF**: NPTH, NPTH, F.Cu at (111.6, 141.9)
- added REF**: NPTH, NPTH, F.Cu at (140.8, 120.9)
- added REF**: NPTH, NPTH, F.Cu at (110.6, 141.9)
- added REF**: NPTH, NPTH, F.Cu at (109.6, 141.9)
- added REF**: NPTH, NPTH, F.Cu at (108.6, 141.9)
- added REF**: NPTH, NPTH, F.Cu at (81.6, 141.9)
- added REF**: NPTH, NPTH, F.Cu at (80.6, 141.9)
- added REF**: NPTH, NPTH, F.Cu at (79.6, 141.9)
- added REF**: NPTH, NPTH, F.Cu at (78.6, 141.9)
- added REF**: NPTH, NPTH, F.Cu at (108.6, 112.3)
- added REF**: NPTH, NPTH, F.Cu at (109.6, 112.3)
- added REF**: NPTH, NPTH, F.Cu at (110.6, 112.3)
- added REF**: NPTH, NPTH, F.Cu at (140.8, 121.9)
- added REF**: NPTH, NPTH, F.Cu at (111.6, 112.3)
- added REF**: NPTH, NPTH, F.Cu at (78.6, 112.3)
- added REF**: NPTH, NPTH, F.Cu at (79.6, 112.3)
- added REF**: NPTH, NPTH, F.Cu at (80.6, 112.3)
- added REF**: NPTH, NPTH, F.Cu at (81.6, 112.3)
- added REF**: NPTH, NPTH, F.Cu at (111.6, 110.5)
- added REF**: NPTH, NPTH, F.Cu at (110.6, 110.5)
- added REF**: NPTH, NPTH, F.Cu at (109.6, 110.5)
- added REF**: NPTH, NPTH, F.Cu at (108.6, 110.5)
- added REF**: NPTH, NPTH, F.Cu at (81.6, 110.5)
- added REF**: NPTH, NPTH, F.Cu at (140.8, 122.9)
- added REF**: NPTH, NPTH, F.Cu at (80.6, 110.5)
- added REF**: NPTH, NPTH, F.Cu at (79.6, 110.5)
- added REF**: NPTH, NPTH, F.Cu at (78.6, 110.5)
- added REF**: NPTH, NPTH, F.Cu at (108.6, 80.8)
- added REF**: NPTH, NPTH, F.Cu at (109.6, 80.8)
- added REF**: NPTH, NPTH, F.Cu at (110.6, 80.8)
- added REF**: NPTH, NPTH, F.Cu at (111.6, 80.8)
- added REF**: NPTH, NPTH, F.Cu at (78.6, 80.8)
- added REF**: NPTH, NPTH, F.Cu at (79.6, 80.8)
- added REF**: NPTH, NPTH, F.Cu at (80.6, 80.8)
- added REF**: NPTH, NPTH, F.Cu at (140.8, 123.9)
- added REF**: NPTH, NPTH, F.Cu at (81.6, 80.8)
- added REF**: NPTH, NPTH, F.Cu at (111.6, 79.0)
- added REF**: NPTH, NPTH, F.Cu at (110.6, 79.0)
- added REF**: NPTH, NPTH, F.Cu at (109.6, 79.0)
- added REF**: NPTH, NPTH, F.Cu at (108.6, 79.0)
- added REF**: NPTH, NPTH, F.Cu at (81.6, 79.0)
- added REF**: NPTH, NPTH, F.Cu at (80.6, 79.0)
- added REF**: NPTH, NPTH, F.Cu at (79.6, 79.0)
- added REF**: NPTH, NPTH, F.Cu at (78.6, 79.0)
- added REF**: NPTH, NPTH, F.Cu at (108.6, 49.4)
- added REF**: NPTH, NPTH, F.Cu at (49.4, 133.4)
- added REF**: NPTH, NPTH, F.Cu at (109.6, 49.4)
- added REF**: NPTH, NPTH, F.Cu at (110.6, 49.4)
- added REF**: NPTH, NPTH, F.Cu at (111.6, 49.4)
- added REF**: NPTH, NPTH, F.Cu at (78.6, 49.4)
- added REF**: NPTH, NPTH, F.Cu at (79.6, 49.4)
- added REF**: NPTH, NPTH, F.Cu at (80.6, 49.4)
- added REF**: NPTH, NPTH, F.Cu at (81.6, 49.4)
- added SW1: RST, PTS636:PTS636 SM25F SMTR LFS, F.Cu at (73.6, 120.3)
- added SW1: RST, PTS636:PTS636 SM25F SMTR LFS, F.Cu at (73.6, 88.8)
- added SW1: RST, PTS636:PTS636 SM25F SMTR LFS, F.Cu at (73.6, 57.4)
- added U3: MIC5219-5.0YMM, Package_SO:MSOP-8_3x3mm_P0.65mm, F.Cu at (80.9, 124.8)
- added U3: MIC5219-5.0YMM, Package_SO:MSOP-8_3x3mm_P0.65mm, F.Cu at (80.9, 93.4)
- added U3: MIC5219-5.0YMM, Package_SO:MSOP-8_3x3mm_P0.65mm, F.Cu at (80.9, 61.9)
- added U4: LM27762, Package_SON:WSON-12-1EP_3x2mm_P0.5mm_EP1x2.65_ThermalVias, F.Cu at (107.3, 123.9)
- added U4: LM27762, Package_SON:WSON-12-1EP_3x2mm_P0.5mm_EP1x2.65_ThermalVias, F.Cu at (107.3, 92.5)
- added U4: LM27762, Package_SON:WSON-12-1EP_3x2mm_P0.5mm_EP1x2.65_ThermalVias, F.Cu at (107.3, 61.0)
- added U5: TPS60501DGS, Package_SO:MSOP-10_3x3mm_P0.5mm, F.Cu at (107.2, 132.2)
- added U5: TPS60501DGS, Package_SO:MSOP-10_3x3mm_P0.5mm, F.Cu at (107.2, 100.8)
- added U5: TPS60501DGS, Package_SO:MSOP-10_3x3mm_P0.5mm, F.Cu at (107.2, 69.3)
- added U7: BQ24074RGT, Package_DFN_QFN:VQFN-16-1EP_3x3mm_P0.5mm_EP1.6x1.6mm, F.Cu at (67.7, 130.9)
- added U7: BQ24074RGT, Package_DFN_QFN:VQFN-16-1EP_3x3mm_P0.5mm_EP1.6x1.6mm, F.Cu at (67.7, 99.5)
- added U7: BQ24074RGT, Package_DFN_QFN:VQFN-16-1EP_3x3mm_P0.5mm_EP1.6x1.6mm, F.Cu at (67.7, 68.0)
- added U8: BQ27441DRZR-G1B, Package_SON:Texas_S-PDSO-N12, F.Cu at (72.9, 129.5)
- added U8: BQ27441DRZR-G1B, Package_SON:Texas_S-PDSO-N12, F.Cu at (72.9, 98.1)
- added U8: BQ27441DRZR-G1B, Package_SON:Texas_S-PDSO-N12, F.Cu at (72.9, 66.6)
- added Y1: 32.768, Crystal:Crystal_SMD_2012-2Pin_2.0x1.2mm, F.Cu at (81.8, 131.5)
- added Y1: 32.768, Crystal:Crystal_SMD_2012-2Pin_2.0x1.2mm, F.Cu at (81.8, 100.0)
- added Y1: 32.768, Crystal:Crystal_SMD_2012-2Pin_2.0x1.2mm, F.Cu at (81.8, 68.6)
- U1 (x3): moved to F.Cu
- turned U1 to 90 degrees (x3)
Routing:
- net Board_1-RST: track 116.0 -> 57.5 mm, vias 4 -> 3
- net Board_2-RST: track 116.0 -> 57.5 mm, vias 4 -> 3
- net Board_3-RST: track 116.0 -> 57.5 mm, vias 4 -> 3
- net Board_2-AREF: track 39.7 -> 79.1 mm, vias 1 -> 2
- net Board_3-AREF: track 39.7 -> 79.1 mm, vias 1 -> 2
- net Board_1-AREF: track 39.7 -> 79.1 mm, vias 1 -> 2
- net Board_2-NEOPIXEL_DOUT: track 41.2 -> 76.0 mm, vias 2 -> 1
- net Board_1-NEOPIXEL_DOUT: track 41.2 -> 76.0 mm, vias 2 -> 1
- net Board_3-NEOPIXEL_DOUT: track 41.2 -> 76.0 mm, vias 2 -> 1
- net Board_2-GND: track 48.5 -> 21.7 mm, vias 81 -> 54
- net Board_1-GND: track 48.5 -> 21.7 mm, vias 81 -> 54
- net Board_3-GND: track 48.5 -> 21.7 mm, vias 81 -> 54
- net Board_2-8[MI]: track 100.8 -> 75.1 mm, vias 2 -> 4
- net Board_1-8[MI]: track 100.8 -> 75.1 mm, vias 2 -> 4
- net Board_3-8[MI]: track 100.8 -> 75.1 mm, vias 2 -> 4
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Other:
- outline, holes or cut-outs redrawn
- board text added: "BAT+"
- board text added: "BAT-"
- board text added: "CAN"
- board text added: "QWIIC"
